File: Solar-Panel-Z/SolarCellZ.kicad_sch (KiCad schematic)
At the start: 62 parts, among them J1 XF2M-1015-1A, Q1 IRLML2803, U1 NDS8434, U2 Value, U3 Value

Commit message: Finished Cleanup
Parts:
- U1: footprint custom-footprints:NDS8434 -> misc-circuits:NDS8434
Connections:
- net SOLAR_OUT is gone; now on net VSOLAR_FULL: TP1.1
Changed lines of the file:
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@@
     )
   )
-  (global_label "SOLAR_OUT" (shape bidirectional) (at 191.516 127.254 270) (fields_autoplaced)
+  (global_label "VSOLAR_FULL" (shape bidirectional) (at 191.516 127.254 270) (fields_autoplaced)
     (effects (font (size 1.27 1.27)) (justify right))
-    (property "Intersheet References" "${INTERSHEET_REFS}" (id 0) (at 235.966 133.604 0)
-      (effects (font (size 1.27 1.27)) hide)
+    (property "Intersheet References" "${INTERSHEET_REFS}" (id 0) (at 191.4366 142.0363 90)
+      (effects (font (size 1.27 1.27)) (justify right) hide)
     )
   )
@@
       (effects (font (size 1.27 1.27)) (justify left bottom))
     )
-    (property "Footprint" "custom-footprints:NDS8434" (id 2) (at 298.45 149.606 0)
+    (property "Footprint" "misc-circuits:NDS8434" (id 2) (at 298.45 149.606 0)
       (effects (font (size 1.27 1.27)) (justify left bottom) hide)
     )
@@
     )
     (path "/00000000-0000-0000-0000-00005db28c34"
-      (reference "U1") (unit 1) (value "NDS8434") (footprint "custom-footprints:NDS8434")
+      (reference "U1") (unit 1) (value "NDS8434") (footprint "misc-circuits:NDS8434")
     )
     (path "/6a21efa6-5663-4456-9e7c-e2692e923ecf"
