File: Solar-Panel-Minus-Z/SolarCell-Z.kicad_sch (KiCad schematic)
At the start: 66 parts, among them J1 XF2M-1015-1A, J2 U.FL-R-SMT-1, Q1 IRLML2803, U1 NDS8434, U2 Value, U3 Value, U4 TTB12G51-Balun

Commit message: Done with X, +/-Y, and +Z. TODO: -Z
Parts:
- H1, H2: footprint MountingHole:MountingHole_2.2mm_M2_Pad -> misc-circuits:Antenna Pad
Changed lines of the file:
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@@
       (effects (font (size 1.27 1.27)) (justify left) hide)
     )
-    (property "Footprint" "MountingHole:MountingHole_2.2mm_M2_Pad" (id 2) (at 143.764 176.53 0)
+    (property "Footprint" "misc-circuits:Antenna Pad" (id 2) (at 143.764 176.53 0)
       (effects (font (size 1.27 1.27)) hide)
     )
@@
       (effects (font (size 1.27 1.27)) (justify left) hide)
     )
-    (property "Footprint" "MountingHole:MountingHole_2.2mm_M2_Pad" (id 2) (at 143.764 186.69 0)
+    (property "Footprint" "misc-circuits:Antenna Pad" (id 2) (at 143.764 186.69 0)
       (effects (font (size 1.27 1.27)) hide)
     )
@@
     )
     (path "/20966b2d-14ff-4a15-8dcd-402836f98cb5"
-      (reference "H1") (unit 1) (value "MountingHole_Pad") (footprint "MountingHole:MountingHole_2.2mm_M2_Pad")
+      (reference "H1") (unit 1) (value "MountingHole_Pad") (footprint "misc-circuits:Antenna Pad")
     )
     (path "/e3fffc42-3290-4abc-87ee-001b481bfcd6"
-      (reference "H2") (unit 1) (value "MountingHole_Pad") (footprint "MountingHole:MountingHole_2.2mm_M2_Pad")
+      (reference "H2") (unit 1) (value "MountingHole_Pad") (footprint "misc-circuits:Antenna Pad")
     )
     (path "/f21bef62-2cc3-43f9-99b8-7d46dc07b791"

Commit message: -Z board changes
Parts:
- removed SC3, SC6: SolarCell, SolarCellParts:KXOB25-05X3F, symbol SolarCellParts:SolarCell_Small
- added JP2: Jumper, SolarCellParts:Burn-Wire-Rotated, symbol misc-circuits-cache:Device_Jumper
- renumbered SC4 to SC3, SC5 to SC4, SC7 to SC5, SC8 to SC6
Connections:
- net GND: now also JP2.2
- net VBURN: now also JP2.1
Other:
- moved on the sheet: JP1
