File: Solar-Panel-Y-/Solar-Panel-Y-.kicad_pcb (KiCad board)
At the start: 6 copper layers, 64 x 58 mm, 83 parts, among them J1 FTS-105-01-L-DV-A, J2 BM02B-SRSS-TB, Q1 BSS138DWQ-7, Q2 MBT2222ADW1T1, Q3 BSS138DWQ-7, Q4 MBT2222ADW1T1, SW1 SW_SPDT, SW2 SW_SPDT, U1 BQ25570RGRR, U2 TSL2561

Commit message: Moved Charging connector, added text
Parts:
- moved J2 14.0 mm to (75.5, 71.3)
- moved D3 0.10 mm to (89.3, 60.4)
Routing:
- net BATT_P_SW: track 47.4 -> 56.2 mm
- net BATT_N_SW: track 54.2 -> 49.7 mm
Other:
- outline, holes or cut-outs redrawn
- board text added: "Cable Pinout 1.BATT_N_SW 2.BATT_P_SW 3.BATT_P 4.3V3 5.GND 6.SCL3 7.COIL_P 8.SDA3 9.COIL_N 10.VUSB"
- board text added: "charge at 4.2V 850mA CV/CC"
- board text removed: "Cable Pinout 1.BATT_P 2.BATT_N 3.SDA 4.SCL 5.BURN 6.3V3 7.GND 8.GND 9.COIL_N 10.COIL_P"
Changed lines of the file:
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@@
   )
   (footprint "Capacitor_SMD:C_0402_1005Metric" (layer "B.Cu")
-    (at 96.13802 68.1785 90)
+    (at 96.1136 68.1785 90)
     (descr "Capacitor SMD 0402 (1005 Metric), square (rectangular) end terminal, IPC_7351 nominal, (Body size source: IPC-SM-782 page 76, https://www.pcb-3d.com/wordpress/wp-content/uploads/ipc-sm-782a_amendment_1_and_2.pdf), generated with kicad-footprint-generator")
     (tags "capacitor")
@@
   )
   (footprint "Connector_JST:JST_SH_BM02B-SRSS-TB_1x02-1MP_P1.00mm_Vertical" (layer "B.Cu")
-    (at 75.4888 57.300012 -90)
+    (at 75.4888 71.300012 -90)
     (descr "JST SH series connector, BM02B-SRSS-TB (http://www.jst-mfg.com/product/pdf/eng/eSH.pdf), generated with kicad-footprint-generator")
     (tags "connector JST SH side entry")
@@
   )
   (footprint "solarpanels:MICROSMP" (layer "B.Cu")
-    (at 89.35 60.45)
+    (at 89.35 60.3504)
     (descr "MicroSMP")
     (tags "Schottky Diode")
@@
     (property "Sheetname" "")
     (attr smd)
-    (fp_text reference "D3" (at 2.15 0 90) (layer "B.SilkS")
+    (fp_text reference "D3" (at 0.0072 -0.9652 180) (layer "B.SilkS")
       (effects (font (size 0.381 0.381) (thickness 0.0762)) (justify mirror))
     )
@@
   (gr_line (start 72.8 93.3) (end 136.775 93.3) (layer "Edge.Cuts") (width 0.1))
   (gr_line (start 72.8 35.3) (end 72.8 93.3) (layer "Edge.Cuts") (width 0.1))
-  (gr_circle (center 100.617208 62.617208) (end 105.7 62.6) (layer "Edge.Cuts") (width 0.1) (fill none))
+  (gr_circle (center 100.617208 62.617208) (end 105.867208 62.617208) (layer "Edge.Cuts") (width 0.1) (fill none))
   (gr_line (start 136.775 35.3) (end 136.775 93.3) (layer "Edge.Cuts") (width 0.1))
   (gr_line (start 136.775 35.3) (end 72.8 35.3) (layer "Edge.Cuts") (width 0.1))
@@
     (effects (font (size 0.635 0.635) (thickness 0.1016)) (justify mirror))
   )
+  (gr_text "+" (at 77.5716 68.4784 90) (layer "B.SilkS")
+    (effects (font (size 1.5 1.5) (thickness 0.3)) (justify mirror))
+  )
   (gr_text "VBAT\n" (at 107.3912 63.627) (layer "B.SilkS")
     (effects (font (size 0.635 0.635) (thickness 0.1016)) (justify mirror))
   )
-  (gr_text "Cable Pinout\n1.BATT_P\n2.BATT_N\n3.SDA\n4.SCL\n5.BURN\n6.3V3\n7.GND\n8.GND\n9.COIL_N\n10.COIL_P" (at 95.1738 50.9524) (layer "B.SilkS")
+  (gr_text "-" (at 77.5208 74.0664 90) (layer "B.SilkS")
+    (effects (font (size 1.5 1.5) (thickness 0.3)) (justify mirror))
+  )
+  (gr_text "Cable Pinout\n1.BATT_N_SW\n2.BATT_P_SW\n3.BATT_P\n4.3V3\n5.GND\n6.SCL3\n7.COIL_P\n8.SDA3\n9.COIL_N\n10.VUSB" (at 119.5324 51.435) (layer "B.SilkS")
     (effects (font (size 0.635 0.635) (thickness 0.1016)) (justify left mirror))
   )
+  (gr_text "charge at 4.2V 850mA CV/CC" (at 78.994 71.2978 270) (layer "B.SilkS")
+    (effects (font (size 0.635 0.635) (thickness 0.1016)) (justify mirror))
+  )
   (gr_text "JLCJLCJLCJLC" (at 133.2484 78.1812 90) (layer "F.SilkS")
     (effects (font (size 0.9 0.9) (thickness 0.15)))
@@
     (pts (xy 72.8 93.3) (xy 72.8 35.3))
     (height -3.6866)
-    (gr_text "2283.4646 mils" (at 67.9634 64.3 90) (layer "Dwgs.User")
+    (gr_text "58.0000 mm" (at 67.9634 64.3 90) (layer "Dwgs.User")
       (effects (font (size 1 1) (thickness 0.15)))
     )
@@
     (pts (xy 72.8 35.3) (xy 136.775 35.3))
     (height -3.727799)
-    (gr_text "2518.7008 mils" (at 104.7875 30.422201) (layer "Dwgs.User")
+    (gr_text "63.9750 mm" (at 104.7875 30.422201) (layer "Dwgs.User")
       (effects (font (size 1 1) (thickness 0.15)))
     )
@@
   (segment (start 96.5 77) (end 96.5 77.61152) (width 0.254) (layer "B.Cu") (net 2))
   (via (at 88.75 64.35) (size 0.6) (drill 0.3) (layers "F.Cu" "B.Cu") (net 3))
-  (segment (start 88.75 64.35) (end 93 68.6) (width 0.508) (layer "In3.Cu") (net 3))
-  (segment (start 105.55 68.6) (end 107.4 66.75) (width 0.508) (layer "In3.Cu") (net 3))
-  (segment (start 93 68.6) (end 105.55 68.6) (width 0.508) (layer "In3.Cu") (net 3))
-  (segment (start 97.12802 67.6685) (end 96.13802 68.6585) (width 0.254) (layer "B.Cu") (net 3))
+  (segment (start 88.75 64.35) (end 93 68.6) (width 0.508) (layer "In2.Cu") (net 3))
+  (segment (start 105.55 68.6) (end 107.4 66.75) (width 0.508) (layer "In2.Cu") (net 3))
+  (segment (start 93 68.6) (end 105.55 68.6) (width 0.508) (layer "In2.Cu") (net 3))
+  (segment (start 97.13802 67.6685) (end 96.14802 68.6585) (width 0.254) (layer "B.Cu") (net 3))
   (segment (start 89.23802 64.88802) (end 88.7 64.35) (width 0.508) (layer "B.Cu") (net 3))
   (segment (start 88.75 64.35) (end 86.83952 64.35) (width 0.508) (layer "B.Cu") (net 3))
   (segment (start 89.23802 66.59895) (end 89.23802 64.88802) (width 0.508) (layer "B.Cu") (net 3))
+  (segment (start 96.14802 68.6585) (end 96.1136 68.6585) (width 0.254) (layer "B.Cu") (net 3))
   (segment (start 98.12 69.255357) (end 98.12 68.65) (width 0.254) (layer "B.Cu") (net 4))
   (segment (start 97.467344 70.44916) (end 97.467344 69.908013) (width 0.254) (layer "B.Cu") (net 4))
@@
   (segment (start 87.5216 78.26035) (end 87.5216 79.7785) (width 0.508) (layer "B.Cu") (net 7))
   (via (at 88.7 62.3) (size 0.6) (drill 0.3) (layers "F.Cu" "B.Cu") (net 9))
-  (segment (start 88.7 62.3) (end 88.7 60.45) (width 0.508) (layer "B.Cu") (net 9))
+  (segment (start 88.7 62.3) (end 88.7 60.3504) (width 0.508) (layer "B.Cu") (net 9))
   (via (at 110.45 72.7) (size 0.6) (drill 0.3) (layers "F.Cu" "B.Cu") (net 10))
   (via (at 117.72775 82.005) (size 0.6) (drill 0.3) (layers "F.Cu" "B.Cu") (net 10))
@@
   (segment (start 111.75 64.3) (end 111.75 66.59) (width 0.254) (layer "B.Cu") (net 30))
   (segment (start 121.11 70.7) (end 121.11 71.16) (width 0.254) (layer "B.Cu") (net 30))
-  (via (at 80.6958 56.7944) (size 0.6096) (drill 0.3048) (layers "F.Cu" "B.Cu") (net 31))
-  (segment (start 82.169 55.3212) (end 103.407997 55.3212) (width 0.508) (layer "In3.Cu") (net 31))
-  (segment (start 103.407997 55.3212) (end 105.342004 53.387193) (width 0.508) (layer "In3.Cu") (net 31))
-  (segment (start 80.6958 56.7944) (end 82.169 55.3212) (width 0.508) (layer "In3.Cu") (net 31))
-  (segment (start 115.528 63.573189) (end 105.342004 53.387193) (width 0.762) (layer "B.Cu") (net 31))
-  (segment (start 80.6902 56.8) (end 80.6958 56.7944) (width 0.508) (layer "B.Cu") (net 31))
-  (segment (start 115.528 66.622) (end 115.528 63.573189) (width 0.762) (layer "B.Cu") (net 31))
-  (segment (start 76.8138 56.8) (end 80.6902 56.8) (width 0.508) (layer "B.Cu") (net 31))
-  (via (at 80.6958 57.8104) (size 0.6096) (drill 0.3048) (layers "F.Cu" "B.Cu") (net 32))
-  (segment (start 95.6564 72.7456) (end 102.887602 72.7456) (width 0.508) (layer "In2.Cu") (net 32))
+  (via (at 80.6916 70.7842) (size 0.6096) (drill 0.3048) (layers "F.Cu" "B.Cu") (net 31))
+  (segment (start 86.6648 64.811) (end 86.6648 61.3156) (width 0.508) (layer "In3.Cu") (net 31))
+  (segment (start 80.6916 70.7842) (end 86.6648 64.811) (width 0.508) (layer "In3.Cu") (net 31))
+  (segment (start 86.6648 61.3156) (end 92.2528 55.7276) (width 0.508) (layer "In3.Cu") (net 31))
+  (segment (start 103.001597 55.7276) (end 105.342004 53.387193) (width 0.508) (layer "In3.Cu") (net 31))
+  (segment (start 92.2528 55.7276) (end 103.001597 55.7276) (width 0.508) (layer "In3.Cu") (net 31))
+  (segment (start 76.824012 70.7898) (end 80.686 70.7898) (width 0.508) (layer "B.Cu") (net 31))
+  (segment (start 80.686 70.7898) (end 80.6916 70.7842) (width 0.508) (layer "B.Cu") (net 31))
+  (segment (start 115.528 61.9848) (end 106.930393 53.387193) (width 0.762) (layer "B.Cu") (net 31))
+  (segment (start 106.930393 53.387193) (end 105.342004 53.387193) (width 0.762) (layer "B.Cu") (net 31))
+  (segment (start 115.528 66.622) (end 115.528 61.9848) (width 0.762) (layer "B.Cu") (net 31))
+  (segment (start 76.8138 70.800012) (end 76.824012 70.7898) (width 0.508) (layer "B.Cu") (net 31))
+  (via (at 80.6916 71.8002) (size 0.6096) (drill 0.3048) (layers "F.Cu" "B.Cu") (net 32))
   (segment (start 102.887602 72.7456) (end 105.342004 75.200002) (width 0.508) (layer "In2.Cu") (net 32))
-  (segment (start 80.6958 57.8104) (end 80.7212 57.8104) (width 0.508) (layer "In2.Cu") (net 32))
-  (segment (start 80.7212 57.8104) (end 95.6564 72.7456) (width 0.508) (layer "In2.Cu") (net 32))
+  (segment (start 94.1832 70.1548) (end 96.774 72.7456) (width 0.508) (layer "In2.Cu") (net 32))
+  (segment (start 80.8538 71.8002) (end 82.4992 70.1548) (width 0.508) (layer "In2.Cu") (net 32))
+  (segment (start 96.774 72.7456) (end 102.887602 72.7456) (width 0.508) (layer "In2.Cu") (net 32))
+  (segment (start 80.6916 71.8002) (end 80.8538 71.8002) (width 0.508) (layer "In2.Cu") (net 32))
+  (segment (start 82.4992 70.1548) (end 94.1832 70.1548) (width 0.508) (layer "In2.Cu") (net 32))
+  (segment (start 80.6812 71.7898) (end 80.6916 71.8002) (width 0.508) (layer "B.Cu") (net 32))
   (segment (start 110.871 78.3336) (end 107.737402 75.200002) (width 0.762) (layer "B.Cu") (net 32))
+  (segment (start 76.824012 71.7898) (end 80.6812 71.7898) (width 0.508) (layer "B.Cu") (net 32))
   (segment (start 107.737402 75.200002) (end 105.342004 75.200002) (width 0.762) (layer "B.Cu") (net 32))
   (segment (start 115.528 70.692) (end 115.528 77.131) (width 0.762) (layer "B.Cu") (net 32))
+  (segment (start 76.8138 71.800012) (end 76.824012 71.7898) (width 0.508) (layer "B.Cu") (net 32))
   (segment (start 114.3254 78.3336) (end 110.871 78.3336) (width 0.762) (layer "B.Cu") (net 32))
-  (segment (start 80.6854 57.8) (end 80.6958 57.8104) (width 0.508) (layer "B.Cu") (net 32))
-  (segment (start 76.8138 57.8) (end 80.6854 57.8) (width 0.508) (layer "B.Cu") (net 32))
   (segment (start 115.528 77.131) (end 114.3254 78.3336) (width 0.762) (layer "B.Cu") (net 32))
   (segment (start 120.31 65.11) (end 120.05 64.85) (width 0.254) (layer "B.Cu") (net 34))

Commit message: New Y- Layout
Parts:
- added SC3: SolarCell_Small, solarpanels:KXOB25-05X3F, F.Cu at (122.2, 53.8)
- added SC7: SolarCell_Small, solarpanels:KXOB25-05X3F, F.Cu at (87.4, 53.8)
- moved C10 48.4 mm to (123.7, 49.1), turned to -90 degrees
- moved D2 44.7 mm to (120.8, 48.7), turned to 0 degrees
- moved C11 41.7 mm to (118.2, 48.2), turned to 90 degrees
- moved L2 39.3 mm to (120.4, 52.3), turned to 90 degrees
- moved R16 39.2 mm to (123.7, 58.9), turned to -90 degrees
- moved R15 38.0 mm to (123.7, 61.9), turned to 90 degrees
- moved U2 37.7 mm to (87.3, 50.1), turned to 0 degrees
- moved C7 37.2 mm to (121.7, 56.4), turned to 90 degrees
- moved C2 36.9 mm to (123.3, 64.1), turned to 0 degrees
- moved C9 34.2 mm to (120.0, 56.4), turned to 90 degrees
- moved C8 34.1 mm to (114.1, 49.5), turned to 90 degrees
- moved C6 33.0 mm to (113.1, 49.5), turned to 90 degrees
- moved L1 32.1 mm to (120.4, 60.4), turned to 90 degrees
- moved D3 31.9 mm to (120.3, 68.1), turned to 180 degrees
- moved C13 31.0 mm to (89.6, 70.3)
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Routing:
- net /VSOLAR_FULL: track 23.9 -> 39.5 mm, vias 4 -> 8
- net BATT_P: track 31.8 -> 47.3 mm
- net SDA3: track 21.5 -> 37.0 mm
- net SCL3: track 17.4 -> 32.6 mm
- net Net-(D3-Pad1): track 1.95 -> 14.3 mm
- net BATT_P_SW: track 56.2 -> 65.6 mm, vias 1 -> 2
- net SDA_LS: track 23.5 -> 29.0 mm
- net VBAT: track 43.9 -> 39.5 mm
- net GND: track 13.6 -> 9.38 mm, vias 8 -> 10
- net SCL_LS: track 14.2 -> 17.1 mm, vias 1 -> 2
- net Net-(R1-Pad1): track 7.70 -> 10.6 mm
- net COIL_P: track 13.6 -> 11.1 mm
- net COIL_N: track 17.6 -> 15.2 mm
- net VOUT_EN: track 9.60 -> 11.8 mm
- net +3V3: track 25.1 -> 23.0 mm
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