File: Solar-Panel-X/Solar-Panel-X.kicad_sch (KiCad schematic)
At the start: 73 parts, among them J1 FTS-105-01-L-DV-A, Q1 BSS138DWQ-7, Q2 MBT2222ADW1T1, Q3 BSS138DWQ-7, Q4 MBT2222ADW1T1, U1 BQ25570RGRR, U2 TSL2561

Commit message: Finish 6 Layer panel versions
Parts:
- C10, C11, C12, C13, C2, C3, C4, C6, C7, C8, C9: footprint Capacitor_SMD:C_0402_1005Metric -> Capacitor_SMD:C_0603_1608Metric
- J1: footprint batteryboard:FTS-105-XX-YY-DV-A -> solarpanels:SAMTEC-FTS-105-01-X-DV-A
- R10, R11, R12, R13, R16, R17, R18, R3, R5, R6, R7, R8, R9: footprint Resistor_SMD:R_0402_1005Metric -> Resistor_SMD:R_0603_1608Metric
- R14, R15: value 0 -> DNI; footprint Resistor_SMD:R_0402_1005Metric -> Resistor_SMD:R_0603_1608Metric
- R19: renamed from R22; value 0 -> DNI; footprint Resistor_SMD:R_0402_1005Metric -> Resistor_SMD:R_0603_1608Metric
- R20: renamed from R23; value 0 -> DNI; footprint Resistor_SMD:R_0402_1005Metric -> Resistor_SMD:R_0603_1608Metric
- R21: renamed from R20; footprint Resistor_SMD:R_0402_1005Metric -> Resistor_SMD:R_0603_1608Metric
- R22: renamed from R21; footprint Resistor_SMD:R_0402_1005Metric -> Resistor_SMD:R_0603_1608Metric
- R23: renamed from R24; footprint Resistor_SMD:R_0402_1005Metric -> Resistor_SMD:R_0603_1608Metric
- R24: renamed from R25; footprint Resistor_SMD:R_0402_1005Metric -> Resistor_SMD:R_0603_1608Metric
- R25: renamed from R26; footprint Resistor_SMD:R_0402_1005Metric -> Resistor_SMD:R_0603_1608Metric
- R26: renamed from R27; footprint Resistor_SMD:R_0402_1005Metric -> Resistor_SMD:R_0603_1608Metric
- R27: renamed from R28; footprint Resistor_SMD:R_0402_1005Metric -> Resistor_SMD:R_0603_1608Metric
- R28: renamed from R29; footprint Resistor_SMD:R_0402_1005Metric -> Resistor_SMD:R_0603_1608Metric
- R29: renamed from R30; footprint Resistor_SMD:R_0402_1005Metric -> Resistor_SMD:R_0603_1608Metric
- R30: renamed from R31; footprint Resistor_SMD:R_0402_1005Metric -> Resistor_SMD:R_0603_1608Metric
- R4: renamed from R19; footprint Resistor_SMD:R_0402_1005Metric -> Resistor_SMD:R_0603_1608Metric
- renumbered SC5 to SC1, SC6 to SC2, SC7 to SC3, SC8 to SC4, SC1 to SC5, SC2 to SC6, SC3 to SC7, SC4 to SC8
Connections:
- net BURN2 is gone; now on net GND: J1.4 (Pin_4)
- net VUSB is gone; now on net BATT_P: J1.10 (Pin_10)
- net SCL2 renamed SCL
- net SDA2 renamed SDA
