File: Solar-Panel-Y- (4L)/Solar-Panel-Y-.kicad_pcb (KiCad board)
At the start: 4 copper layers, 64 x 58 mm, 87 parts, among them J1 FTS-107-01-X-DV-A, J2 BM02B-SRSS-TB, Q1 NX3008NBKS, Q2 MBT2222ADW1T1, Q3 NX3008NBKS, Q4 MBT2222ADW1T1, SW1 D2F-L2-A1, SW2 D2F-L2-A, U1 BQ25570RGRR, U2 OPT4001, U3 MAX40200AUK

Commit message: Updated Rev to B3/03
Other:
- board text added: "Rev B3/03"
- board text removed: "Rev B3/02"
Changed lines of the file:
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@@
     (effects (font (size 0.635 0.635) (thickness 0.1016)))
   )
-  (gr_text "Rev B3/02" (at 105.686402 87.69) (layer "B.Mask")
+  (gr_text "Rev B3/03" (at 105.686402 87.69) (layer "B.Mask")
     (effects (font (size 0.635 0.635) (thickness 0.1524)) (justify mirror))
   )

Commit message: Exported stuff
Routing:
- net /coil: track 7475.5 -> 7477.1 mm
Other:
- outline, holes or cut-outs redrawn
